Commit message: adding wingtip projection visualization

File: fly_model/fly.urdf (robot description, URDF)
Before this commit: robot fly, 10 links, 9 joints
Links:
- link thorax: geometry collision mesh filename=thorax.dae; visual mesh filename=thorax.dae
- link wingL: mass 0.01 -> 0.001
- link wingR: mass 0.01 -> 0.001
